File: PCB/SENTINEL Mark II - Quest.kicad_pcb (KiCad board)
At the start: 2 copper layers, 111 parts, among them J1 POWER, J10 External, J11 USB_B_Mini, J2 Conn_01x03, J3 Conn_01x04, J4 Conn_01x03, J5 Conn_01x04, J6 Conn_01x04, J7 SERVO1, J8 SERVO2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

Commit message: Add new file
edge-cut.cdr
Parts:
- moved C1 79.8 mm to (192.8, 110.2)
- moved C10 79.8 mm to (201.6, 109.8)
- moved C12 79.8 mm to (191.5, 90.5)
- moved C3 79.8 mm to (198.5, 106.9)
- moved C7 79.8 mm to (205.3, 102.3)
- moved D3 79.8 mm to (194.6, 103.1)
- moved FB1 79.8 mm to (190.6, 119.1)
- moved L1 79.8 mm to (185.9, 105.3)
- moved Q1 79.8 mm to (200.9, 103.1)
- moved R16 79.8 mm to (190.8, 136.6)
- moved R2 79.8 mm to (200.2, 116.1)
- moved R5 79.8 mm to (200.2, 113.2)
- moved CM4 79.8 mm to (115.2, 93.4)
- moved DM2 79.8 mm to (124.4, 91.6)
- moved C11 79.8 mm to (196.3, 83.7)
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
Commit message: KICAD
Parts:
- moved RESET1 241.9 mm to (402.8, 93.9)
- moved J3 241.9 mm to (382.4, 104.9)
- moved J4 241.9 mm to (391.7, 92.7)
- moved J6 241.9 mm to (382.4, 92.7)
- moved R11 241.9 mm to (358.2, 120.3)
- moved SW1 241.9 mm to (393.5, 103.6)
- moved SW4 241.9 mm to (397.3, 110.7)
- moved J2 241.9 mm to (396.3, 92.7)
- moved J5 241.9 mm to (387.0, 92.7)
- moved LCD1 241.9 mm to (361.8, 92.3)
- moved R10 241.9 mm to (353.8, 120.3)
- moved SW2 241.9 mm to (401.9, 103.6)
- moved SW3 241.9 mm to (388.9, 110.7)
- moved SW5 241.9 mm to (392.7, 117.9)
- moved SW6 241.9 mm to (405.7, 110.7)
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Routing:
- net (no net): vias 0 -> 4
Other:
- board outline added: 96.7 x 64.2 mm
