File: PCB/Power Supply.sch (KiCad schematic (older format))
At the start: 26 parts, among them J1 POWER, Q1 AO3401, U1 LD1117S33TR, U2 MP2307

Commit message: Footprint Assigned
Parts:
- C1, C10, C2, C3, C4, C5, C6, C7, C8, C9: footprint (none) -> Capacitor_SMD:C_0805_2012Metric
- D1, D3: footprint (none) -> Diode_SMD:D_SMA
- D2: footprint (none) -> Diode_SMD:D_SOD-123
- FB1: footprint (none) -> Inductor_SMD:L_0805_2012Metric
- J1: footprint (none) -> Connector_PinHeader_2.54mm:PinHeader_1x02_P2.54mm_Vertical
- L1: footprint (none) -> Inductor_SMD:L_7.3x7.3_H3.5
- R1, R2, R3, R4, R5, R6: footprint (none) -> Resistor_SMD:R_0805_2012Metric
- S1: footprint (none) -> Kicad Library:switch_slide_2.54
- U2: footprint SOIC8N_EP_MNP -> Kicad Library:MP2307
Changed lines of the file:
@@
 F 0 "U2" H 7500 3500 60  0000 C CNN
 F 1 "MP2307" H 7500 3400 60  0000 C CNN
-F 2 "SOIC8N_EP_MNP" H 7500 3840 60  0001 C CNN
+F 2 "Kicad Library:MP2307" H 7500 3840 60  0001 C CNN
 F 3 "" H 6700 3600 60  0000 C CNN
 	1    6700 3600
@@
 F 0 "C5" H 5800 3875 50  0000 L CNN
 F 1 "100nF" H 5675 3800 50  0000 L CNN
-F 2 "" H 6038 3700 50  0001 C CNN
+F 2 "Capacitor_SMD:C_0805_2012Metric" H 6038 3700 50  0001 C CNN
 F 3 "~" H 6000 3850 50  0001 C CNN
 	1    6000 3850
@@
 F 0 "C6" V 6350 3600 50  0000 C CNN
 F 1 "100nF" V 6425 3600 50  0000 C CNN
-F 2 "" H 6588 3450 50  0001 C CNN
+F 2 "Capacitor_SMD:C_0805_2012Metric" H 6588 3450 50  0001 C CNN
 F 3 "~" H 6550 3600 50  0001 C CNN
 	1    6550 3600
@@
 F 0 "R2" H 6500 4250 50  0000 C CNN
 F 1 "100K" V 6600 4300 50  0000 C CNN
-F 2 "" V 6530 4300 50  0001 C CNN
+F 2 "Resistor_SMD:R_0805_2012Metric" V 6530 4300 50  0001 C CNN
 F 3 "~" H 6600 4300 50  0001 C CNN
 	1    6600 4300
@@
 F 0 "L1" V 6450 3325 50  0000 R CNN
 F 1 "10uH/4A" V 6350 3450 50  0000 R CNN
-F 2 "" H 6400 3025 50  0001 C CNN
+F 2 "Inductor_SMD:L_7.3x7.3_H3.5" H 6400 3025 50  0001 C CNN
 F 3 "~" H 6400 3025 50  0001 C CNN
 	1    6400 3025
@@
 F 0 "C4" H 5350 3875 50  0000 L CNN
 F 1 "22uF" H 5275 3800 50  0000 L CNN
-F 2 "" H 5588 3700 50  0001 C CNN
+F 2 "Capacitor_SMD:C_0805_2012Metric" H 5588 3700 50  0001 C CNN
 F 3 "~" H 5550 3850 50  0001 C CNN
 	1    5550 3850
@@
 F 0 "C7" H 6715 2971 50  0000 L CNN
 F 1 "33uF" H 6715 2880 50  0000 L CNN
-F 2 "" H 6638 2775 50  0001 C CNN
+F 2 "Capacitor_SMD:C_0805_2012Metric" H 6638 2775 50  0001 C CNN
 F 3 "~" H 6600 2925 50  0001 C CNN
 	1    6600 2925
@@
 F 0 "C8" H 7165 2971 50  0000 L CNN
 F 1 "33uF" H 7165 2880 50  0000 L CNN
-F 2 "" H 7088 2775 50  0001 C CNN
+F 2 "Capacitor_SMD:C_0805_2012Metric" H 7088 2775 50  0001 C CNN
 F 3 "~" H 7050 2925 50  0001 C CNN
 	1    7050 2925
@@
 F 0 "R6" V 8925 4050 50  0000 R CNN
 F 1 "10K" V 9025 4075 50  0000 R CNN
-F 2 "" V 8955 4000 50  0001 C CNN
+F 2 "Resistor_SMD:R_0805_2012Metric" V 8955 4000 50  0001 C CNN
 F 3 "~" H 9025 4000 50  0001 C CNN
 	1    9025 4000
@@
 F 0 "R5" H 8550 4100 50  0000 R CNN
 F 1 "2K2" V 8600 4225 50  0000 R CNN
-F 2 "" V 8530 4150 50  0001 C CNN
+F 2 "Resistor_SMD:R_0805_2012Metric" V 8530 4150 50  0001 C CNN
 F 3 "~" H 8600 4150 50  0001 C CNN
 	1    8600 4150
@@
 F 0 "R3" H 6500 4550 50  0000 C CNN
 F 1 "33K" V 6600 4600 50  0000 C CNN
-F 2 "" V 6530 4600 50  0001 C CNN
+F 2 "Resistor_SMD:R_0805_2012Metric" V 6530 4600 50  0001 C CNN
 F 3 "~" H 6600 4600 50  0001 C CNN
 	1    6600 4600
@@
 F 0 "C9" H 8375 3500 50  0000 C CNN
 F 1 "100nF" H 8300 3575 50  0000 C CNN
-F 2 "" H 8563 3400 50  0001 C CNN
+F 2 "Capacitor_SMD:C_0805_2012Metric" H 8563 3400 50  0001 C CNN
 F 3 "~" H 8525 3550 50  0001 C CNN
 	1    8525 3550
@@
 F 0 "R4" V 8525 3950 50  0000 R CNN
 F 1 "6K8" V 8600 3975 50  0000 R CNN
-F 2 "" V 8530 3900 50  0001 C CNN
+F 2 "Resistor_SMD:R_0805_2012Metric" V 8530 3900 50  0001 C CNN
 F 3 "~" H 8600 3900 50  0001 C CNN
 	1    8600 3900
@@
 F 0 "D3" V 6425 3775 50  0000 L CNN
 F 1 "SS54" V 6500 3700 50  0000 L CNN
-F 2 "" H 6400 3950 50  0001 C CNN
+F 2 "Diode_SMD:D_SMA" H 6400 3950 50  0001 C CNN
 F 3 "~" H 6400 3950 50  0001 C CNN
 	1    6400 3950
@@
 F 0 "C10" H 8775 3725 50  0000 C CNN
 F 1 "3.9nF" H 8725 3800 50  0000 C CNN
-F 2 "" H 8963 3600 50  0001 C CNN
+F 2 "Capacitor_SMD:C_0805_2012Metric" H 8963 3600 50  0001 C CNN
 F 3 "~" H 8925 3750 50  0001 C CNN
 	1    8925 3750
@@
 F 0 "S1" H 3800 3885 50  0000 C CNN
 F 1 "ON-OFF" H 3800 3794 50  0000 C CNN
-F 2 "" H 3800 3600 50  0001 C CNN
+F 2 "Kicad Library:switch_slide_2.54" H 3800 3600 50  0001 C CNN
 F 3 "~" H 3800 3600 50  0001 C CNN
 	1    3800 3600
@@
 F 0 "C2" H 5015 5071 50  0000 L CNN
 F 1 "22uF" H 5015 4980 50  0000 L CNN
-F 2 "" H 4938 4875 50  0001 C CNN
+F 2 "Capacitor_SMD:C_0805_2012Metric" H 4938 4875 50  0001 C CNN
 F 3 "~" H 4900 5025 50  0001 C CNN
 	1    4900 5025
@@
 F 0 "FB1" V 3301 4875 50  0000 C CNN
 F 1 "1A" V 3392 4875 50  0000 C CNN
-F 2 "" V 3505 4875 50  0001 C CNN
+F 2 "Inductor_SMD:L_0805_2012Metric" V 3505 4875 50  0001 C CNN
 F 3 "~" H 3575 4875 50  0001 C CNN
 	1    3575 4875
@@
 F 0 "C1" H 3965 5071 50  0000 L CNN
 F 1 "100nF" H 3965 4980 50  0000 L CNN
-F 2 "" H 3888 4875 50  0001 C CNN
+F 2 "Capacitor_SMD:C_0805_2012Metric" H 3888 4875 50  0001 C CNN
 F 3 "~" H 3850 5025 50  0001 C CNN
 	1    3850 5025
@@
 F 0 "J1" H 3168 3375 50  0000 C CNN
 F 1 "POWER" H 3168 3466 50  0000 C CNN
-F 2 "" H 3250 3700 50  0001 C CNN
+F 2 "Connector_PinHeader_2.54mm:PinHeader_1x02_P2.54mm_Vertical" H 3250 3700 50  0001 C CNN
 F 3 "~" H 3250 3700 50  0001 C CNN
 	1    3250 3700
@@
 F 0 "C3" H 4925 3875 50  0000 L CNN
 F 1 "22uF" H 4850 3800 50  0000 L CNN
-F 2 "" H 5163 3700 50  0001 C CNN
+F 2 "Capacitor_SMD:C_0805_2012Metric" H 5163 3700 50  0001 C CNN
 F 3 "~" H 5125 3850 50  0001 C CNN
 	1    5125 3850
@@
 F 0 "R1" V 5100 2775 50  0000 C CNN
 F 1 "10K" V 5200 2775 50  0000 C CNN
-F 2 "" V 5130 2775 50  0001 C CNN
+F 2 "Resistor_SMD:R_0805_2012Metric" V 5130 2775 50  0001 C CNN
 F 3 "~" H 5200 2775 50  0001 C CNN
 	1    5200 2775
@@
 F 0 "D2" V 5429 2554 50  0000 L CNN
 F 1 "5.1V" V 5520 2554 50  0000 L CNN
-F 2 "" H 5475 2475 50  0001 C CNN
+F 2 "Diode_SMD:D_SOD-123" H 5475 2475 50  0001 C CNN
 F 3 "~" H 5475 2475 50  0001 C CNN
 	1    5475 2475
@@
 F 0 "D1" H 4325 2509 50  0000 C CNN
 F 1 "SS34" H 4325 2600 50  0000 C CNN
-F 2 "" H 4325 2725 50  0001 C CNN
+F 2 "Diode_SMD:D_SMA" H 4325 2725 50  0001 C CNN
 F 3 "~" H 4325 2725 50  0001 C CNN
 	1    4325 2725

Commit message: Circuit fix (Kicad)
Parts:
- removed D2: 5.1V, Diode_SMD:D_SOD-123, symbol Device:D_Zener_ALT
- removed Q1: AO3401, Package_TO_SOT_SMD:SOT-23, symbol Transistor_FET:AO3401A
- removed R1: 10K, Resistor_SMD:R_0805_2012Metric, symbol Device:R
Connections:
- net GND: now also R4.2; no longer C10.2
- net at U2.6 (COMP): now also C10.2; no longer R4.2
Other:
- note removed: "A"
- note removed: "B"
- note removed: "Reverse polarity protection, choose one: A or B"
- moved on the sheet: C10, D1, J1, R4, S1
Changed lines of the file:
@@
 L Device:R R4
 U 1 1 5F5ED02C
-P 8600 3900
-F 0 "R4" V 8525 3950 50  0000 R CNN
-F 1 "6K8" V 8600 3975 50  0000 R CNN
-F 2 "Resistor_SMD:R_0805_2012Metric" V 8530 3900 50  0001 C CNN
-F 3 "~" H 8600 3900 50  0001 C CNN
-	1    8600 3900
-	0    1    1    0
+P 8925 3750
+F 0 "R4" V 8850 3800 50  0000 R CNN
+F 1 "6K8" V 8925 3825 50  0000 R CNN
+F 2 "Resistor_SMD:R_0805_2012Metric" V 8855 3750 50  0001 C CNN
+F 3 "~" H 8925 3750 50  0001 C CNN
+	1    8925 3750
+	-1   0    0    1
 $EndComp
 Wire Wire Line
@@
 L Device:C C10
 U 1 1 5F5F536F
-P 8925 3750
-F 0 "C10" H 8775 3725 50  0000 C CNN
-F 1 "3.9nF" H 8725 3800 50  0000 C CNN
-F 2 "Capacitor_SMD:C_0805_2012Metric" H 8963 3600 50  0001 C CNN
-F 3 "~" H 8925 3750 50  0001 C CNN
-	1    8925 3750
-	-1   0    0    1
+P 8600 3900
+F 0 "C10" V 8400 3950 50  0000 C CNN
+F 1 "3.9nF" V 8475 3975 50  0000 C CNN
+F 2 "Capacitor_SMD:C_0805_2012Metric" H 8638 3750 50  0001 C CNN
+F 3 "~" H 8600 3900 50  0001 C CNN
+	1    8600 3900
+	0    1    1    0
 $EndComp
 Wire Wire Line
@@
 	1    0    0    -1
 $EndComp
-Text Label 4575 3700 0    50   ~ 0
+Text Label 4100 3700 0    50   ~ 0
 12V
 $Comp
 L power:GND #PWR01
 U 1 1 5F621368
-P 3450 3700
-F 0 "#PWR01" H 3450 3450 50  0001 C CNN
-F 1 "GND" H 3450 3550 50  0000 C CNN
-F 2 "" H 3450 3700 50  0001 C CNN
-F 3 "" H 3450 3700 50  0001 C CNN
-	1    3450 3700
+P 2850 3700
+F 0 "#PWR01" H 2850 3450 50  0001 C CNN
+F 1 "GND" H 2850 3550 50  0000 C CNN
+F 2 "" H 2850 3700 50  0001 C CNN
+F 3 "" H 2850 3700 50  0001 C CNN
+	1    2850 3700
 	1    0    0    -1
 $EndComp
@@
 	6400 4250 6400 4100
 Wire Wire Line
-	3450 3600 3600 3600
-Text Notes 4000 4100 0    50   ~ 0
+	2850 3600 3000 3600
+Text Notes 3400 4100 0    50   ~ 0
 3A Fuse Trace:\n1.4mm width\n1oz thickness
 Wire Notes Line
@@
 $EndComp
 Wire Wire Line
-	4000 3700 4075 3700
-Wire Wire Line
-	4075 3700 4075 3825
-Wire Wire Line
-	4075 3825 4150 3825
-Wire Wire Line
-	4150 3825 4150 3575
-Wire Wire Line
-	4150 3575 4225 3575
-Wire Wire Line
-	4225 3575 4225 3825
-Wire Wire Line
-	4225 3825 4300 3825
-Wire Wire Line
-	4300 3825 4300 3575
-Wire Wire Line
-	4300 3575 4375 3575
-Wire Wire Line
-	4375 3575 4375 3825
-Wire Wire Line
-	4375 3825 4450 3825
-Wire Wire Line
-	4450 3825 4450 3700
-Wire Wire Line
-	4450 3700 4575 3700
+	3400 3700 3475 3700
+Wire Wire Line
+	3475 3700 3475 3825
+Wire Wire Line
+	3475 3825 3550 3825
+Wire Wire Line
+	3550 3825 3550 3575
+Wire Wire Line
+	3550 3575 3625 3575
+Wire Wire Line
+	3625 3575 3625 3825
+Wire Wire Line
+	3625 3825 3700 3825
+Wire Wire Line
+	3700 3825 3700 3575
+Wire Wire Line
+	3700 3575 3775 3575
+Wire Wire Line
+	3775 3575 3775 3825
+Wire Wire Line
+	3775 3825 3850 3825
+Wire Wire Line
+	3850 3825 3850 3700
 $Comp
 L Connector_Generic:Conn_01x02 J1
 U 1 1 5F61FDC3
-P 3250 3700
-F 0 "J1" H 3168 3375 50  0000 C CNN
-F 1 "POWER" H 3168 3466 50  0000 C CNN
-F 2 "Connector_PinHeader_2.54mm:PinHeader_1x02_P2.54mm_Vertical" H 3250 3700 50  0001 C CNN
-F 3 "~" H 3250 3700 50  0001 C CNN
-	1    3250 3700
+P 2650 3700
+F 0 "J1" H 2568 3375 50  0000 C CNN
+F 1 "POWER" H 2568 3466 50  0000 C CNN
+F 2 "Connector_PinHeader_2.54mm:PinHeader_1x02_P2.54mm_Vertical" H 2650 3700 50  0001 C CNN
+F 3 "~" H 2650 3700 50  0001 C CNN
+	1    2650 3700
 	-1   0    0    1
 $EndComp
@@
 $EndComp
 $Comp
-L Transistor_FET:AO3401A QM?
-U 1 1 5F686A99
-P 5200 2425
-AR Path="/5F60FE64/5F686A99" Ref="QM?"  Part="1"
-AR Path="/5F592C3C/5F686A99" Ref="Q1"  Part="1"
-F 0 "Q1" V 5500 2425 50  0000 C CNN
-F 1 "AO3401" V 5425 2425 50  0000 C CNN
-F 2 "Package_TO_SOT_SMD:SOT-23" H 5400 2350 50  0001 L CIN
-F 3 "http://www.aosmd.com/pdfs/datasheet/AO3401A.pdf" H 5200 2425 50  0001 L CNN
-	1    5200 2425
-	0    -1   -1   0
-$EndComp
-$Comp
-L Device:R RM?
-U 1 1 5F686AA0
-P 5200 2775
-AR Path="/5F60FE64/5F686AA0" Ref="RM?"  Part="1"
-AR Path="/5F592C3C/5F686AA0" Ref="R1"  Part="1"
-F 0 "R1" V 5100 2775 50  0000 C CNN
-F 1 "10K" V 5200 2775 50  0000 C CNN
-F 2 "Resistor_SMD:R_0805_2012Metric" V 5130 2775 50  0001 C CNN
-F 3 "~" H 5200 2775 50  0001 C CNN
-	1    5200 2775
-	-1   0    0    1
-$EndComp
-$Comp
-L Device:D_Zener_ALT DM?
-U 1 1 5F686AA6
-P 5475 2475
-AR Path="/5F60FE64/5F686AA6" Ref="DM?"  Part="1"
-AR Path="/5F592C3C/5F686AA6" Ref="D2"  Part="1"
-F 0 "D2" V 5429 2554 50  0000 L CNN
-F 1 "5.1V" V 5520 2554 50  0000 L CNN
-F 2 "Diode_SMD:D_SOD-123" H 5475 2475 50  0001 C CNN
-F 3 "~" H 5475 2475 50  0001 C CNN
-	1    5475 2475
-	0    1    1    0
-$EndComp
-Wire Wire Line
-	5475 2625 5200 2625
-Connection ~ 5200 2625
-Wire Wire Line
-	5400 2325 5475 2325
-Text Label 5725 2325 0    50   ~ 0
-Vin
-$Comp
-L power:GND #PWR?
-U 1 1 5F686AB0
-P 5200 2925
-AR Path="/5F60FE64/5F686AB0" Ref="#PWR?"  Part="1"
-AR Path="/5F592C3C/5F686AB0" Ref="#PWR03"  Part="1"
-F 0 "#PWR03" H 5200 2675 50  0001 C CNN
-F 1 "GND" H 5200 2775 50  0000 C CNN
-F 2 "" H 5200 2925 50  0001 C CNN
-F 3 "" H 5200 2925 50  0001 C CNN
-	1    5200 2925
-	1    0    0    -1
-$EndComp
-Wire Notes Line
-	3950 3125 3950 2075
-Text Notes 3975 2175 0    50   ~ 10
-A
-Text Notes 4725 2175 0    50   ~ 10
-B
-Text Notes 3975 2050 0    50   ~ 0
-Reverse polarity protection, choose one: A or B
-Wire Wire Line
-	5725 2325 5475 2325
-Connection ~ 5475 2325
-Wire Notes Line
-	5850 2075 5850 3125
-Wire Notes Line
-	5850 3125 3950 3125
-Wire Notes Line
-	3950 2075 5850 2075
-$Comp
 L Device:D_Schottky_ALT D1
 U 1 1 5F68F386
-P 4325 2725
-F 0 "D1" H 4325 2509 50  0000 C CNN
-F 1 "SS34" H 4325 2600 50  0000 C CNN
-F 2 "Diode_SMD:D_SMA" H 4325 2725 50  0001 C CNN
-F 3 "~" H 4325 2725 50  0001 C CNN
-	1    4325 2725
+P 4675 3700
+F 0 "D1" H 4675 3484 50  0000 C CNN
+F 1 "SS34" H 4675 3575 50  0000 C CNN
+F 2 "Diode_SMD:D_SMA" H 4675 3700 50  0001 C CNN
+F 3 "~" H 4675 3700 50  0001 C CNN
+	1    4675 3700
 	-1   0    0    1
 $EndComp
-Text Label 4175 2725 2    50   ~ 0
-12V
-Text Label 4475 2725 0    50   ~ 0
-Vin
 Text Label 5125 3700 2    50   ~ 0
 Vin
-Text Label 5000 2325 2    50   ~ 0
-12V
-Wire Notes Line
-	4850 3650 4850 3425
-Wire Notes Line
-	4850 3425 4700 3425
-Wire Notes Line
-	4700 2075 4700 3425
 $Comp
 L Switch:SW_SPDT S1
 U 1 1 5F6168FF
-P 3800 3600
-F 0 "S1" H 3800 3885 50  0000 C CNN
-F 1 "ON-OFF" H 3800 3794 50  0000 C CNN
-F 2 "Kicad Library:switch_slide_2.54" H 3800 3600 50  0001 C CNN
-F 3 "~" H 3800 3600 50  0001 C CNN
-	1    3800 3600
-	1    0    0    -1
-$EndComp
+P 3200 3600
+F 0 "S1" H 3200 3885 50  0000 C CNN
+F 1 "ON-OFF" H 3200 3794 50  0000 C CNN
+F 2 "Kicad Library:switch_slide_2.54" H 3200 3600 50  0001 C CNN
+F 3 "~" H 3200 3600 50  0001 C CNN
+	1    3200 3600
+	1    0    0    -1
+$EndComp
+Wire Wire Line
+	4825 3700 5125 3700
+Connection ~ 5125 3700
+Wire Wire Line
+	3850 3700 4525 3700
 $EndSCHEMATC
