File: PCB/USB.sch (KiCad schematic (older format))
At the start: 12 parts, among them J11 USB_B_Mini, Q2 MMBT3906

Commit message: Footprint Assigned
Parts:
- C19, C20, C21: footprint (none) -> Capacitor_SMD:C_0805_2012Metric
- D5: footprint (none) -> Diode_SMD:D_SMA
- FB5: footprint (none) -> Inductor_SMD:L_0805_2012Metric
- J11: footprint (none) -> Connector_USB:USB_Mini-B_Lumberg_2486_01_Horizontal
- JP2: footprint (none) -> Jumper:SolderJumper-2_P1.3mm_Open_RoundedPad1.0x1.5mm
- R13, R14, R15, R16: footprint (none) -> Resistor_SMD:R_0805_2012Metric
Changed lines of the file:
@@
 F 0 "J11" H 6750 3775 50  0000 C CNN
 F 1 "USB_B_Mini" H 6600 3875 50  0000 C CNN
-F 2 "" H 7175 3700 50  0001 C CNN
+F 2 "Connector_USB:USB_Mini-B_Lumberg_2486_01_Horizontal" H 7175 3700 50  0001 C CNN
 F 3 "~" H 7175 3700 50  0001 C CNN
 	1    7025 3750
@@
 F 0 "FB5" H 6500 3150 50  0000 C CNN
 F 1 "1A" H 6525 3075 50  0000 C CNN
-F 2 "" V 6655 3100 50  0001 C CNN
+F 2 "Inductor_SMD:L_0805_2012Metric" V 6655 3100 50  0001 C CNN
 F 3 "~" H 6725 3100 50  0001 C CNN
 	1    6725 3100
@@
 F 0 "R15" V 6375 3700 50  0000 L CNN
 F 1 "0-22" V 6450 3650 50  0000 L CNN
-F 2 "" V 6380 3750 50  0001 C CNN
+F 2 "Resistor_SMD:R_0805_2012Metric" V 6380 3750 50  0001 C CNN
 F 3 "~" H 6450 3750 50  0001 C CNN
 	1    6450 3750
@@
 F 0 "R16" V 6525 3800 50  0000 L CNN
 F 1 "0-22" V 6450 3750 50  0000 L CNN
-F 2 "" V 6380 3850 50  0001 C CNN
+F 2 "Resistor_SMD:R_0805_2012Metric" V 6380 3850 50  0001 C CNN
 F 3 "~" H 6450 3850 50  0001 C CNN
 	1    6450 3850
@@
 F 0 "C20" V 5975 4250 50  0000 C CNN
 F 1 "33pF" V 6050 4250 50  0000 C CNN
-F 2 "" H 6213 4100 50  0001 C CNN
+F 2 "Capacitor_SMD:C_0805_2012Metric" H 6213 4100 50  0001 C CNN
 F 3 "~" H 6175 4250 50  0001 C CNN
 	1    6175 4250
@@
 F 0 "C19" V 5625 4250 50  0000 C CNN
 F 1 "33pF" V 5700 4250 50  0000 C CNN
-F 2 "" H 5863 4100 50  0001 C CNN
+F 2 "Capacitor_SMD:C_0805_2012Metric" H 5863 4100 50  0001 C CNN
 F 3 "~" H 5825 4250 50  0001 C CNN
 	1    5825 4250
@@
 F 0 "C21" V 6650 2750 50  0000 L CNN
 F 1 "100nF" V 6725 2700 50  0000 L CNN
-F 2 "" H 6913 2650 50  0001 C CNN
+F 2 "Capacitor_SMD:C_0805_2012Metric" H 6913 2650 50  0001 C CNN
 F 3 "~" H 6875 2800 50  0001 C CNN
 	1    6875 2800
@@
 F 0 "R14" H 5875 3325 50  0000 L CNN
 F 1 "1K5" V 5825 3200 50  0000 L CNN
-F 2 "" V 5755 3275 50  0001 C CNN
+F 2 "Resistor_SMD:R_0805_2012Metric" V 5755 3275 50  0001 C CNN
 F 3 "~" H 5825 3275 50  0001 C CNN
 	1    5825 3275
@@
 F 0 "R13" V 5300 2925 50  0000 C CNN
 F 1 "1K" V 5375 2925 50  0000 C CNN
-F 2 "" V 5305 2925 50  0001 C CNN
+F 2 "Resistor_SMD:R_0805_2012Metric" V 5305 2925 50  0001 C CNN
 F 3 "~" H 5375 2925 50  0001 C CNN
 	1    5375 2925
@@
 F 0 "JP2" V 5779 3668 50  0000 L CNN
 F 1 "DISC" V 5870 3668 50  0000 L CNN
-F 2 "" H 5825 3600 50  0001 C CNN
+F 2 "Jumper:SolderJumper-2_P1.3mm_Open_RoundedPad1.0x1.5mm" H 5825 3600 50  0001 C CNN
 F 3 "~" H 5825 3600 50  0001 C CNN
 	1    5825 3600
@@
 F 0 "D5" H 6575 3016 50  0000 C CNN
 F 1 "SS14" H 6575 2925 50  0000 C CNN
-F 2 "" H 6575 2800 50  0001 C CNN
+F 2 "Diode_SMD:D_SMA" H 6575 2800 50  0001 C CNN
 F 3 "~" H 6575 2800 50  0001 C CNN
 	1    6575 2800

Commit message: Circuit fix (Kicad)
Connections:
- net D-: now reaches J11.2 (D-), R16.2
- net D+: now reaches J11.3 (D+), R15.2
- net USBDM renamed USBD-
- net USBDP renamed USBD+
Changed lines of the file:
@@
 	6375 2800 6425 2800
 Text HLabel 4625 3750 0    50   Input ~ 0
-USBDP
+USBD+
 Text HLabel 4625 3850 0    50   Output ~ 0
-USBDM
+USBD-
 $Comp
 L Device:D_Schottky_ALT D5
@@
 $EndComp
 Connection ~ 6725 2800
+Text Label 6600 3750 0    50   ~ 0
+D+
+Text Label 6600 3850 0    50   ~ 0
+D-
 $EndSCHEMATC
