File: Schematic/USB.sch (KiCad schematic (older format))
At the start: 12 parts, among them J11 USB_B_Mini, Q2 MMBT3906

Commit message: Schematic update
Parts:
- J11: symbol Connector:USB_B_Mini -> SENTINEL-Mark-II---Quest-rescue:USB_B_Mini-Connector
Changed lines of the file:
@@
 $EndDescr
 $Comp
-L Connector:USB_B_Mini J?
+L SENTINEL-Mark-II---Quest-rescue:USB_B_Mini-Connector J?
 U 1 1 5F6C87FB
 P 7025 3750
